File: TMC5160HV.kicad_sch (KiCad schematic)
At the start: 28 parts, among them J1 825433-4, J2 825433-8, J3 825433-8, Q1 STL8DN10LF3, Q2 STL8DN10LF3, Q3 STL8DN10LF3, Q4 STL8DN10LF3, U1 TMC5160-TA

Commit message: 1206 for caps and 0603 for resistors
Parts:
- C1, C10, C11, C12, C2, C3, C4, C5, C6, C7, C8, C9: footprint (none) -> Capacitor_SMD:C_1206_3216Metric
- Q1, Q2, Q3, Q4: footprint STL50DN6F7 -> lib:STL50DN6F7
- R1, R2, R3, R4, R5, R6, R7, R8: footprint (none) -> Resistor_SMD:R_0603_1608Metric
